Commit message: 重新设计深度相机，可继续原来的建图

File: src/gazebo_pkg/urdf/waking_robot.xacro (robot description, xacro)
@@ -4,5 +4,5 @@
 	<xacro:property name="radius_wheel" value="0.06" />
 	<xacro:property name="camera_link" value="0.05" />
-        <xacro:property name="PI" value="3.1415926"/>
+  <xacro:property name="PI" value="3.1415926"/>
 	<xacro:macro name="default_inertial" params="mass">
                <inertial>
@@ -86,4 +86,5 @@
 			<origin rpy="0 0 0" xyz="0 0 0"/>
    			<material name="black"/>
+        <color rgba="0 0 0 1"/>
    		</visual>
 		<collision>
@@ -215,6 +216,6 @@
 	<box size="0.05 0.05 0.05"/>
       </geometry>
-      <material name="red">
-	<color rgba="1 0 0 1"/>
+      <material name="blue">
+	<color rgba="0 0 1 1"/>
       </material>
     </visual>
@@ -279,5 +280,5 @@
   <!-- camera_link -->
   <gazebo reference="camera_link">
-    <material>Gazebo/Red</material>
+    <material>Gazebo/Blue</material>
   </gazebo>
   <!-- hokuyo -->
@@ -321,36 +322,38 @@
     </sensor>
   </gazebo>
-  <!-- camera -->
+  <!-- 深度摄像头 -->
   <gazebo reference="camera_link">
-    <sensor type="camera" name="camera1">
+    <sensor type="depth" name="camera_depth_sensor">
       <update_rate>30.0</update_rate>
-      <camera name="head">
-        <horizontal_fov>1.3962634</horizontal_fov>
+      <camera>
+        <horizontal_fov>1.047</horizontal_fov>
         <image>
-          <width>1920</width>
-          <height>1080</height>
+          <width>640</width>
+          <height>480</height>
           <format>R8G8B8</format>
         </image>
         <clip>
-          <near>0.02</near>
-          <far>300</far>
+          <near>0.05</near>
+          <far>5.0</far>
         </clip>
         <noise>
           <type>gaussian</type>
-          <!-- Noise is sampled independently per pixel on each frame.
-               That pixel's noise value is added to each of its color
-               channels, which at that point lie in the range [0,1]. -->
           <mean>0.0</mean>
           <stddev>0.007</stddev>
         </noise>
       </camera>
-      <plugin name="camera_controller" filename="libgazebo_ros_camera.so">
+      <plugin name="camera_depth_controller" filename="libgazebo_ros_depth_camera.so">
         <alwaysOn>true</alwaysOn>
-        <updateRate>0.0</updateRate>
-        <cameraName>/</cameraName>
-        <imageTopicName>cam</imageTopicName>
-        <cameraInfoTopicName>camera_info</cameraInfoTopicName>
+        <updateRate>30.0</updateRate>
+        <cameraName>camera_depth</cameraName>
+        <imageTopicName>camera/depth/image_raw</imageTopicName>
+        <cameraInfoTopicName>camera/depth/camera_info</cameraInfoTopicName>
+        <pointCloudTopicName>camera/depth/points</pointCloudTopicName>
+        <depthImageTopicName>camera/depth/image_depth</depthImageTopicName>
+        <depthImageCameraInfoTopicName>camera/depth/camera_info_depth</depthImageCameraInfoTopicName>
+        <pointCloudCutoff>0.05</pointCloudCutoff>
+        <pointCloudCutoffMax>5.0</pointCloudCutoffMax>
+        <hackBaseline>0.07</hackBaseline>
         <frameName>camera_link</frameName>
-        <hackBaseline>0.07</hackBaseline>
         <distortionK1>0.0</distortionK1>
         <distortionK2>0.0</distortionK2>
@@ -403,43 +406,4 @@
     </gazebo>
 <!-- gazebo插件设置相关结束 -->
-<!-- 深度摄像头
-<joint name="camera_depth_joint" type="fixed">
-  <parent link="base_link"/>
-  <child link="camera_depth_link"/>
-  <origin xyz="0.2 0 0.2" rpy="0 0 0"/>
-</joint>
-<link name="camera_depth_link">
-  <visual>
-    <geometry>
-      <box size="0.05 0.05 0.05"/>
-    </geometry>
-    <material name="black"/>
-  </visual>
-</link>
-<gazebo reference="camera_depth_link">
-  <sensor type="depth" name="camera_depth">
-    <update_rate>30.0</update_rate>
-    <camera>
-      <horizontal_fov>1.047</horizontal_fov>
-      <image>
-        <width>640</width>
-        <height>480</height>
-        <format>R8G8B8</format>
-      </image>
-      <clip>
-        <near>0.05</near>
-        <far>5.0</far>
-      </clip>
-    </camera>
-    <plugin name="camera_depth_controller" filename="libgazebo_ros_depth_camera.so">
-      <alwaysOn>true</alwaysOn>
-      <updateRate>30.0</updateRate>
-      <cameraName>camera_depth</cameraName>
-      <imageTopicName>camera/depth/image_raw</imageTopicName>
-      <cameraInfoTopicName>camera/depth/camera_info</cameraInfoTopicName>
-      <frameName>camera_depth_link</frameName>
-      <pointCloudTopicName>camera/depth/points</pointCloudTopicName>
-    </plugin>
-  </sensor>
-</gazebo> -->
+<!-- 原来的深度摄像头代码已被整合到camera_link中 -->
 </robot>

Commit message: 删除dummy

File: src/gazebo_pkg/urdf/waking_robot.xacro (robot description, xacro)
@@ -14,6 +14,4 @@
                </inertial>
 	</xacro:macro>
-    <link name="dummy">
-    </link>
 	<link name="base_footprint">
    		<visual>
@@ -25,8 +23,4 @@
 		<xacro:default_inertial mass="0.0001"/>
  	</link>
-   <joint name="dummy_joint" type="fixed">
-     <parent link="dummy"/>
-     <child link="base_footprint"/>
-   </joint>
 <!--  	<xacro:include filename="$(find nav_sim)/urdf/robot.gazebo" />  -->
 	<gazebo reference="base_footprint">
@@ -35,8 +29,12 @@
 	</gazebo>
 	<joint name="base_footprint_joint" type="fixed">
-		<origin xyz="0 0 0" />
+		<!-- <origin xyz="0 0 0" />
 		<parent link="base_footprint" />
 		<child link="base_link" />
-	</joint>
+	</joint> -->
+    <origin xyz="0 0 0.06" />  <!-- 当前是0，应该设置为0.06 -->
+    <parent link="base_footprint" />
+    <child link="base_link" />
+</joint>
 	<link name="base_link">
    		<visual>
@@ -338,9 +336,4 @@
           <far>5.0</far>
         </clip>
-        <noise>
-          <type>gaussian</type>
-          <mean>0.0</mean>
-          <stddev>0.007</stddev>
-        </noise>
       </camera>
       <plugin name="camera_depth_controller" filename="libgazebo_ros_depth_camera.so">
@@ -353,18 +346,8 @@
         <depthImageCameraInfoTopicName>depth/camera_info</depthImageCameraInfoTopicName>
         <pointCloudTopicName>depth/points</pointCloudTopicName>
-        <frameName>camera_link</frameName>
+        <frameName>camera_depth_frame</frameName>  <!-- 改为camera_depth_frame -->
         <hackBaseline>0.07</hackBaseline>
         <pointCloudCutoff>0.05</pointCloudCutoff>
         <pointCloudCutoffMax>5.0</pointCloudCutoffMax>
-        <updateRate>30</updateRate>
-        <publishImage>true</publishImage>
-        <publishCameraInfo>true</publishCameraInfo>
-        <publishDepth>true</publishDepth>
-        <publishPointCloud>true</publishPointCloud>
-        <distortionK1>0.0</distortionK1>
-        <distortionK2>0.0</distortionK2>
-        <distortionK3>0.0</distortionK3>
-        <distortionT1>0.0</distortionT1>
-        <distortionT2>0.0</distortionT2>
       </plugin>
     </sensor>
@@ -386,5 +369,5 @@
     <odometryTopic>odom</odometryTopic>
     <odometryFrame>odom</odometryFrame>
-    <robotBaseFrame>dummy</robotBaseFrame>
+    <robotBaseFrame>base_footprint</robotBaseFrame>  <!-- 改为base_footprint -->
     <broadcastTF>1</broadcastTF>
   </plugin>
@@ -413,3 +396,17 @@
 <!-- gazebo插件设置相关结束 -->
 <!-- 原来的深度摄像头代码已被整合到camera_link中 -->
+<!-- Camera depth frame joint -->
+<joint name="camera_depth_joint" type="fixed">
+    <origin xyz="0 0 0" rpy="0 0 0"/>
+    <parent link="camera_link"/>
+    <child link="camera_depth_frame"/>
+</joint>
+<!-- Camera depth frame -->
+<link name="camera_depth_frame">
+    <inertial>
+        <mass value="1e-5" />
+        <origin xyz="0 0 0" rpy="0 0 0"/>
+        <inertia ixx="1e-6" ixy="0" ixz="0" iyy="1e-6" iyz="0" izz="1e-6" />
+    </inertial>
+</link>
 </robot>
